File: pcb/relaymux.kicad_pcb (KiCad board)
At the start: 2 copper layers, 120.4 x 100.4 mm, 60 parts, among them J1 A, J10 B4, J11 USB_C, J12 Debug, J2 A1, J3 A2, J4 A3, J5 A4, J6 B, J7 B1, J8 B2, J9 B3, K1 TQ2SA-5V, K2 TQ2SA-5V, K3 TQ2SA-5V, K4 TQ2SA-5V, K5 TQ2SA-5V, K6 TQ2SA-5V, K7 TQ2SA-5V, K8 TQ2SA-5V, SW1 Cycle, SW2 Boot/Clear, U1 STM32F042F4Px, U2 TBD62783A, U3 TPS2552D, U4 TLV70033_SOT23-5

Commit message: First version of firmware
Parts:
- C2: value 10µF -> N/A
- R11, R12, R14, R15: value 47k -> 75k
- U1: value STM32F042F4Px -> STM32F042F6Px
